File: hardware/pi-crust-plus/design/pi-crust-plus.brd (EAGLE design)
At the start: 13 parts

Commit message: update hardware designs for plus and protohat
update hardware designs for plus and protohat
Other:
- board text added: "Pi Crust Plus"
- board text removed: "Pi Crust B Plus"
