File: hardware/pi-crust-protohat/design/pi-crust-protohat.sch (EAGLE design)
At the start: 13 parts, among them U1 EEPROM24

Commit message: update hardware designs for plus and protohat
update hardware designs for plus and protohat
Connections:
- removed net N$14: JP5.9
- net +5V: now also U$1.N.C.0
- net GND: now also U$1.N.C.5, U$1.N.C.6, U$1.N.C.8
- net GPIO_26: now also JP5.9
Changed lines of the file:
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@@
 <?xml version="1.0" encoding="utf-8"?>
 <!DOCTYPE eagle SYSTEM "eagle.dtd">
-<eagle version="6.5.0">
+<eagle version="7.6.0">
 <drawing>
 <settings>
@@
 <pinref part="U$1" gate="G$1" pin="GND"/>
 </segment>
+<segment>
+<wire x1="73.66" y1="86.36" x2="83.82" y2="86.36" width="0.1524" layer="91"/>
+<label x="83.82" y="86.36" size="1.778" layer="95"/>
+</segment>
+<segment>
+<wire x1="73.66" y1="83.82" x2="83.82" y2="83.82" width="0.1524" layer="91"/>
+<label x="83.82" y="83.82" size="1.778" layer="95"/>
+</segment>
+<segment>
+<wire x1="73.66" y1="78.74" x2="83.82" y2="78.74" width="0.1524" layer="91"/>
+<label x="83.82" y="78.74" size="1.778" layer="95"/>
+</segment>
+<segment>
+<pinref part="U$1" gate="G$1" pin="N.C.5"/>
+<wire x1="76.2" y1="76.2" x2="83.82" y2="76.2" width="0.1524" layer="91"/>
+<label x="83.82" y="76.2" size="1.778" layer="95"/>
+</segment>
+<segment>
+<pinref part="U$1" gate="G$1" pin="N.C.6"/>
+<wire x1="76.2" y1="73.66" x2="83.82" y2="73.66" width="0.1524" layer="91"/>
+<label x="83.82" y="73.66" size="1.778" layer="95"/>
+</segment>
+<segment>
+<wire x1="73.66" y1="71.12" x2="83.82" y2="71.12" width="0.1524" layer="91"/>
+<label x="83.82" y="71.12" size="1.778" layer="95"/>
+</segment>
+<segment>
+<pinref part="U$1" gate="G$1" pin="N.C.8"/>
+<wire x1="76.2" y1="68.58" x2="83.82" y2="68.58" width="0.1524" layer="91"/>
+<label x="83.82" y="68.58" size="1.778" layer="95"/>
+</segment>
 </net>
 <net name="+3V3" class="0">
@@
 <pinref part="U$1" gate="G$1" pin="3V3"/>
 </segment>
+<segment>
+<wire x1="73.66" y1="81.28" x2="83.82" y2="81.28" width="0.1524" layer="91"/>
+<label x="83.82" y="81.28" size="1.778" layer="95"/>
+</segment>
 </net>
 <net name="N$3" class="0">
@@
 <net name="GPIO_26" class="0">
 <segment>
+<pinref part="JP5" gate="A" pin="9"/>
+<wire x1="243.84" y1="76.2" x2="226.06" y2="76.2" width="0.1524" layer="91"/>
+<label x="226.06" y="76.2" size="1.778" layer="95"/>
+</segment>
+<segment>
+<pinref part="U$1" gate="G$1" pin="GPIO26"/>
 <wire x1="45.72" y1="66.04" x2="38.1" y2="66.04" width="0.1524" layer="91"/>
-<pinref part="U$1" gate="G$1" pin="GPIO26"/>
 </segment>
 </net>
@@
 <pinref part="JP6" gate="A" pin="2"/>
 </segment>
-</net>
-<net name="N$14" class="0">
-<segment>
-<pinref part="JP5" gate="A" pin="9"/>
-<wire x1="243.84" y1="76.2" x2="226.06" y2="76.2" width="0.1524" layer="91"/>
-</segment>
-</net>
+<segment>
+<pinref part="U$1" gate="G$1" pin="N.C.0"/>
+<wire x1="76.2" y1="88.9" x2="83.82" y2="88.9" width="0.1524" layer="91"/>
+<label x="83.82" y="88.9" size="1.778" layer="95"/>
+</segment>
+</net>
